File: pico chiptune player.kicad_sch (KiCad schematic)
At the start: 24 parts, among them J1 MicroSD, J2 Speaker Out, SW1 Play / Pause, SW2 Next, SW3 Previous, U1 AY-3-8910, U2 PAM8302AAS, U3 0.96"OLED_I2C

Commit message: Refactor code structure for improved readability and maintainability
Parts:
- removed JP1: SEL_TEST2, Jumper:SolderJumper-3_P2.0mm_Open_TrianglePad1.0x1.5mm, symbol Jumper:Jumper_3_Open
- removed RV1: 20K, symbol Device:R_Potentiometer_Small
- added JP1: Clk Div, Jumper:SolderJumper-2_P1.3mm_Open_TrianglePad1.0x1.5mm, symbol Jumper:Jumper_2_Open
- added RV1: 3224W-1-103E, Potentiometer_SMD:Potentiometer_Bourns_3224W_Vertical, symbol BOURNS_3224W-1-103E:BOURNS_3224W-1-103E
- U2: footprint (none) -> Package_SO:SOIC-8_5.3x5.3mm_P1.27mm
Connections:
- net GND: now also JP1.2 (B), RV1.1
- net at U1.26 (~{CS/Test_2}): now also JP1.1 (A)
- net at U2.3 (IN+): now also RV1.2
- net at C3.2: now also RV1.3
Other:
- moved on the sheet: C2, C3, C4, C5, J2, R4, R5, R6, R7, R8, U1, U2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

Commit message: Refactor schematic and project files: Update active layer, modify visible layers, and add polarized capacitor symbol
- Changed active layer from 5 to 2 in the KiCad project file.
- Updated visible layers in the project file for better visibility.
- Removed unused designators and added a new polarized capacitor symbol in the schematic.
- Introduced properties for the new capacitor symbol including reference, value, footprint, and description.
- Cleaned up the schematic by removing the old unpolarized capacitor symbol.
Parts:
- removed C3: 1uF, Capacitor_SMD:C_0805_2012Metric_Pad1.18x1.45mm_HandSolder, symbol Device:C
- added C3: 1uF, Capacitor_SMD:CP_Elec_3x5.4, symbol Device:C_Polarized
Connections:
- net at C2.1, R4.2, R5.2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: now also C3.1
- net at RV1.3: now also C3.2
Changed lines of the file:
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@@
+	)
+	(symbol
+		(lib_id "Device:C_Polarized")
+		(at 194.31 116.84 90)
+		(unit 1)
+		(body_style 1)
+		(exclude_from_sim no)
+		(in_bom yes)
+		(on_board yes)
+		(in_pos_files yes)
+		(dnp no)
+		(fields_autoplaced yes)
+		(property "Reference" "C3"
+			(at 193.421 109.22 90)
+			(show_name no)
+			(do_not_autoplace no)
+			(effects
+				(font
+					(size 1.27 1.27)
+				)
+			)
+		)
+		(property "Value" "1uF"
+			(at 193.421 111.76 90)
+			(show_name no)
+			(do_not_autoplace no)
+			(effects
+				(font
+					(size 1.27 1.27)
+				)
+			)
+		)
+		(property "Footprint" "Capacitor_SMD:CP_Elec_3x5.4"
+			(at 198.12 115.8748 0)
+			(show_name no)
+			(do_not_autoplace no)
+			(effects
+				(font
+					(size 1.27 1.27)
+				)
+			)
+		)
+		(property "Datasheet" ""
+			(at 194.31 116.84 0)
+			(hide yes)
+			(show_name no)
+			(do_not_autoplace no)
+			(effects
+				(font
+					(size 1.27 1.27)
+				)
+			)
+		)
+		(property "Description" "Polarized capacitor"
+			(at 194.31 116.84 0)
+			(hide yes)
+			(show_name no)
+			(do_not_autoplace no)
+			(effects
+				(font
+					(size 1.27 1.27)
+				)
+			)
+		)
+		(pin "2"
+		)
+		(pin "1"
+		)
+		(instances
+			(project "pico chiptune player"
+				(path "/7838ce79-4aa7-49e0-80b2-fad97ae8a425"
+					(reference "C3")
+					(unit 1)
+				)
+			)
+		)
 	)
 	(symbol
@@
 					(unit 1)
 				)
-			)
-		)
-	)
-	(symbol
-		(lib_id "Device:C")
-		(at 194.31 116.84 90)
-		(unit 1)
-		(body_style 1)
-		(exclude_from_sim no)
-		(in_bom yes)
-		(on_board yes)
-		(in_pos_files yes)
-		(dnp no)
-		(property "Reference" "C3"
-			(at 191.77 115.062 90)
-			(show_name no)
-			(do_not_autoplace no)
-			(effects
-				(font
-					(size 1.27 1.27)
-				)
-			)
-		)
-		(property "Value" "1uF"
-			(at 190.754 118.618 90)
-			(show_name no)
-			(do_not_autoplace no)
-			(effects
-				(font
-					(size 1.27 1.27)
-				)
-			)
-		)
-		(property "Footprint" "Capacitor_SMD:C_0805_2012Metric_Pad1.18x1.45mm_HandSolder"
-			(at 194.31 116.84 0)
-			(hide yes)
-			(show_name no)
-			(do_not_autoplace no)
-			(effects
-				(font
-					(size 1.27 1.27)
-				)
-			)
-		)
-		(property "Datasheet" ""
-			(at 194.31 116.84 0)
-			(show_name no)
-			(do_not_autoplace no)
-			(effects
-				(font
-					(size 1.27 1.27)
-				)
-			)
-		)
-		(property "Description" "Unpolarized capacitor"
-			(at 205.486 133.35 0)
-			(hide yes)
-			(show_name no)
-			(do_not_autoplace no)
-			(effects
-				(font
-					(size 1.27 1.27)
-				)
-			)
-		)
-		(pin "1"
-		)
-		(pin "2"
-		)
-		(instances
-			(project "pico chiptune player"
-				(path "/7838ce79-4aa7-49e0-80b2-fad97ae8a425"
-					(reference "C3")
-					(unit 1)
-				)

Commit message: refactor: remove redundant junctions and update wire connections in schematic
Connections:
- net +5V: no longer U1.27 (BDIR)
- net BDIR: now also U1.27 (BDIR)
Changed lines of the file:
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@@
-	)
-	(junction
-		(at 196.85 69.85)
-		(diameter 0)
-		(color 0 0 0 0)
 	)
 	(junction
@@
 	(wire
 		(pts
-			(xy 196.85 69.85) (xy 196.85 67.31)
+			(xy 196.85 67.31) (xy 196.85 74.93)
 		)
 		(stroke
@@
 	(wire
 		(pts
-			(xy 196.85 74.93) (xy 196.85 69.85)
-		)
-		(stroke
-			(width 0)
-			(type default)
-		)
-	)
-	(wire
-		(pts
 			(xy 222.25 31.75) (xy 222.25 34.29)
 		)
@@
 	(wire
 		(pts
+			(xy 185.42 69.85) (xy 187.96 69.85)
+		)
+		(stroke
+			(width 0)
+			(type default)
+		)
+	)
+	(wire
+		(pts
 			(xy 59.69 157.48) (xy 62.23 157.48)
 		)
@@
 		(pts
 			(xy 185.42 82.55) (xy 187.96 82.55)
-		)
-		(stroke
-			(width 0)
-			(type default)
-		)
-	)
-	(wire
-		(pts
-			(xy 185.42 69.85) (xy 196.85 69.85)
 		)
 		(stroke
@@
 		)
 	)
+	(label "BDIR"
+		(at 187.96 69.85 0)
+		(effects
+			(font
+				(size 1.27 1.27)
+			)
+			(justify left)
+		)
+	)
