File: pico chiptune player.kicad_sch (KiCad schematic)
At the start: 40 parts, among them J2 MicroSD, J3 Speaker_L, J4 Speaker_R, SW1 Play / Pause, SW2 Next, SW3 Previous, U1 YM2149F, U2 0.96"OLED_I2C, U3 PAM8403, U4 YM2149F

Commit message: Refactor code structure for improved readability and maintainability
Parts:
- removed A1: RaspberryPi_Pico 2, TMCu Module:RPi_Pico_SMD_TH, symbol MCU_Module_RaspberryPi_Pico:RaspberryPi_Pico
- added C17, C19: 10uF, Capacitor_SMD:C_0805_2012Metric_Pad1.18x1.45mm_HandSolder, symbol Device:C
- added C18, C24, C25, C26, C27, C28, C29, C30, C31, C33, C34: 100nF, Capacitor_SMD:C_0805_2012Metric_Pad1.18x1.45mm_HandSolder, symbol Device:C
- added C20, C21: 15pF, Capacitor_SMD:C_0805_2012Metric_Pad1.18x1.45mm_HandSolder, symbol Device:C
- added C22, C23: 4.7uF, Capacitor_SMD:C_0805_2012Metric_Pad1.18x1.45mm_HandSolder, symbol Device:C
- added C32: 10nF, Capacitor_SMD:C_0805_2012Metric_Pad1.18x1.45mm_HandSolder, symbol Device:C
- added D1: USBLC6-2SC6, Package_TO_SOT_SMD:SOT-23-6, symbol Power_Protection:USBLC6-2SC6
- added J1: USB_C_5V3A, Connector_USB:USB_C_Receptacle_HRO_TYPE-C-31-M-12, symbol Connector:USB_C_Receptacle_USB2.0_16P
- added L1: 3.3uH, Inductor_SMD:L_1210_3225Metric, symbol Device:L
- added Q1: AO3401A, Package_TO_SOT_SMD:SOT-23, symbol Transistor_FET:AO3401A
- added Q2: 2N7002, Package_TO_SOT_SMD:SOT-23, symbol Transistor_FET:2N7002
- added R14, R15: 470, Resistor_SMD:R_0805_2012Metric_Pad1.20x1.40mm_HandSolder, symbol Device:R
- added R16, R20: 1k, Resistor_SMD:R_0805_2012Metric_Pad1.20x1.40mm_HandSolder, symbol Device:R
- added R17, R18: 27, Resistor_SMD:R_0805_2012Metric_Pad1.20x1.40mm_HandSolder, symbol Device:R
- added R19, R24, R25, R26, R27: 10K, Resistor_SMD:R_0805_2012Metric_Pad1.20x1.40mm_HandSolder, symbol Device:R
- added R21, R22: 5.1k, Resistor_SMD:R_0805_2012Metric_Pad1.20x1.40mm_HandSolder, symbol Device:R
- added R23: 47K, Resistor_SMD:R_0805_2012Metric_Pad1.20x1.40mm_HandSolder, symbol Device:R
- added R28: 100K, Resistor_SMD:R_0805_2012Metric_Pad1.20x1.40mm_HandSolder, symbol Device:R
- added SW4: BOOTSEL, Button_Switch_THT:SW_PUSH_6mm, symbol Switch:SW_Push
- added SW5: RESET, Button_Switch_THT:SW_PUSH_6mm, symbol Switch:SW_Push
- added U5: RP2354A, Package_DFN_QFN:QFN-60-1EP_7x7mm_P0.4mm_EP3.4x3.4mm, symbol MCU_RaspberryPi:RP2354A
- added U6: AMS1117-3.3, Package_TO_SOT_SMD:SOT-223-3_TabPin2, symbol Regulator_Linear:AMS1117-3.3
- added U8, U9: 74HCT4053D, Package_SO:SOIC-16_3.9x9.9mm_P1.27mm, symbol Analog_Switch:CD4053B
- added Y1: 12MHz, Crystal:Crystal_SMD_3225-4Pin_3.2x2.5mm, symbol Device:Crystal_GND24
- C1, C15, C6: footprint Capacitor_SMD:CP_Elec_4x5.4 -> Capacitor_SMD:C_0805_2012Metric_Pad1.18x1.45mm_HandSolder; LCSC Part # C3343 -> C15850
- C11: footprint Capacitor_SMD:CP_Elec_4x5.4 -> Capacitor_SMD:C_0805_2012Metric_Pad1.18x1.45mm_HandSolder
- C2, C7: LCSC Part # C1711 -> C49678
- C4, C5: LCSC Part # C1710 -> C49678
- SW1: LCSC Part # C17513 -> C114217
- SW3: LCSC Part # C12740 -> C114217
Connections:
- net +3.3V: now also C19.1, C22.1, C27.1, C28.1, C29.1, C30.1, R19.1, R23.1, U5.1 (IOVDD), U5.11 (IOVDD), U5.20 (IOVDD), U5.30 (IOVDD), U5.38 (IOVDD), U5.44 (ADC_AVDD), U5.45 (IOVDD), U5.46 (VREG_AVDD), U5.49 (VREG_VIN), U5.53 (USB_OTP_VDD), U5.54 (QSPI_IOVDD), U6.2 (VO)
- net +5V: now also C32.2, C33.1, C34.1, Q1.3 (D), U8.16 (VDD), U9.16 (VDD)
- net BC1: now also U5.12 (GPIO8)
- net BC1_2: now also U5.41 (GPIO27/ADC1)
- net BDIR: now also U5.14 (GPIO10)
- net BDIR2: now also U5.40 (GPIO26/ADC0)
- net DA0: now also U5.2 (GPIO0)
- net DA1: now also U5.3 (GPIO1)
- net DA2: now also U5.4 (GPIO2)
- net DA3: now also U5.5 (GPIO3)
- net DA4: now also U5.7 (GPIO4)
- net DA5: now also U5.8 (GPIO5)
- net DA6: now also U5.9 (GPIO6)
- net DA7: now also U5.10 (GPIO7)
- net GND: now also C17.2, C18.2, C19.2, C20.2, C21.2, C22.2, C23.2, C24.2, C25.2, C26.2, C27.2, C28.2, C29.2, C30.2, C31.2, C33.2, C34.2, D1.2 (GND), J1.A1 (GND), J1.A12 (GND), J1.B1 (GND), J1.B12 (GND), J1.SH (SHIELD), Q2.2 (S), R21.2, R22.2, R24.2, R25.2, R26.2, R27.2, SW4.2, SW5.2, U5.47 (VREG_PGND), U5.61 (GND), U6.1 (GND), U8.6 (INH), U8.7 (VEE), U8.8 (VSS), U9.6 (INH), U9.7 (VEE), U9.8 (VSS), Y1.2 (G), Y1.4 (G)
- net MIX2: now also R15.2, U8.12 (A0), U8.2 (B0), U8.3 (C1), U9.12 (A0); no longer R10.2, R11.2, R9.2
- net OLED_SCL: now also U5.28 (GPIO17)
- net OLED_SDA: now also U5.27 (GPIO16)
- net SD_Amp: now also U5.13 (GPIO9)
- net SD_CLK: now also U5.34 (GPIO22)
- net SD_CMD: now also U5.42 (GPIO28/ADC2)
- net SD_DAT0: now also U5.29 (GPIO18)
- net SD_DAT1: now also U5.31 (GPIO19)
- net SD_DAT2: now also U5.32 (GPIO20)
- net SD_DAT3: now also U5.33 (GPIO21)
- net SW_NEXT: now also U5.17 (GPIO13)
- net SW_PLAY: now also U5.18 (GPIO14)
- net SW_PREV: now also U5.19 (GPIO15)
- net ~{RESET}: now also U5.15 (GPIO11)
- net MIX1: now reaches C3.1, C4.1, R4.2, R8.1
- net MIX1: now also R14.2, U8.4 (C), U9.13 (A1), U9.2 (B0), U9.5 (C0); no longer R5.2, R7.2
- net MCU_CLK: now reaches R2.2
- net MCU_CLK: now also U5.16 (GPIO12)
- new net +1V1: C23.1, C24.1, C25.1, C26.1, L1.2, U5.23 (DVDD), U5.39 (DVDD), U5.50 (VREG_FB), U5.6 (DVDD)
- new net A2_SUM: R9.2, U9.14 (A)
- new net B1_SUM: R5.2, U9.15 (B)
- new net BOOT_BTN: R20.2, SW4.1
- new net C1_SUM: R7.2, U9.4 (C)
- new net MCU_RUN: R19.2, SW5.1, U5.26 (RUN)
- new net MCU_USB_DM: R17.2, U5.51 (USB_DM)
- new net MCU_USB_DP: R18.2, U5.52 (USB_DP)
- new net MIX_C: R14.1, R15.1, U8.1 (B1), U8.13 (A1)
- new net MUX_B_CEN: R25.1, U5.36 (GPIO24), U8.11 (S1)
- new net MUX_C_CEN: R26.1, U5.37 (GPIO25), U8.10 (S2)
- new net MUX_MONO: R27.1, U5.43 (GPIO29/ADC3), U8.9 (S3)
- new net MUX_PAN: R24.1, U5.35 (GPIO23), U9.10 (S2), U9.11 (S1), U9.9 (S3)
- new net NODE_B_PAN: R10.2, U8.14 (A), U9.1 (B1)
- new net NODE_C_PAN: R11.2, U8.15 (B), U9.3 (C1)
- new net PFET_GATE: C32.1, Q1.1 (G), Q2.3 (D), R28.2
- new net QSPI_SS: R20.1, U5.60 (~{QSPI_SS})
- new net SEQ_GATE: C31.1, Q2.1 (G), R23.2
- new net USB_CC1: J1.A5 (CC1), R21.1
- new net USB_CC2: J1.B5 (CC2), R22.1
- new net USB_D+: D1.3 (I/O2), D1.4 (I/O2), J1.A6 (D+), J1.B6 (D+), R18.1
- new net USB_D-: D1.1 (I/O1), D1.6 (I/O1), J1.A7 (D-), J1.B7 (D-), R17.1
- new net VBUS: C17.1, C18.1, D1.5 (VBUS), J1.A4 (VBUS), J1.A9 (VBUS), J1.B4 (VBUS), J1.B9 (VBUS), Q1.2 (S), R28.1, U6.3 (VI)
- new net VREG_LX: L1.1, U5.48 (VREG_LX)
- new net XIN: C20.1, U5.21 (XIN), Y1.1
- new net XOUT: C21.1, R16.2, Y1.3
- new net XOUT_MCU: R16.1, U5.22 (XOUT)
- no-connect marks 44 -> 49

Commit message: Refactor code structure for improved readability and maintainability
Parts:
- C1, C15, C17, C19, C22, C23, C6: footprint Capacitor_SMD:C_0805_2012Metric_Pad1.18x1.45mm_HandSolder -> Capacitor_SMD:C_0805_2012Metric
- C10, C13, C14, C16, C3, C8: footprint Capacitor_SMD:C_0805_2012Metric_Pad1.18x1.45mm_HandSolder -> Capacitor_SMD:C_0402_1005Metric; LCSC Part # C28323 -> C52923
- C11: footprint Capacitor_SMD:C_0805_2012Metric_Pad1.18x1.45mm_HandSolder -> Capacitor_SMD:C_0805_2012Metric; LCSC Part # (none) -> C15850
- C12, C9: footprint Capacitor_SMD:C_0805_2012Metric_Pad1.18x1.45mm_HandSolder -> Capacitor_SMD:C_0402_1005Metric; LCSC Part # (none) -> C307331
- C18, C2, C24, C25, C26, C27, C28, C29, C30, C31, C33, C34, C4, C5, C7: footprint Capacitor_SMD:C_0805_2012Metric_Pad1.18x1.45mm_HandSolder -> Capacitor_SMD:C_0402_1005Metric; LCSC Part # C49678 -> C307331
- C20, C21: footprint Capacitor_SMD:C_0805_2012Metric_Pad1.18x1.45mm_HandSolder -> Capacitor_SMD:C_0402_1005Metric; LCSC Part # C1794 -> C1548
- C32: footprint Capacitor_SMD:C_0805_2012Metric_Pad1.18x1.45mm_HandSolder -> Capacitor_SMD:C_0402_1005Metric; LCSC Part # C1710 -> C15195
- J2: footprint Terence:MicroSD -> Connector_Card:microSD_HC_Hirose_DM3AT-SF-PEJM5; LCSC Part # C479742 -> C114218
- L1: footprint Inductor_SMD:L_1210_3225Metric -> Inductor_SMD:L_Sunlord_MWSA0402S; LCSC Part # C408412 -> C408336
- R1, R13, R19, R24, R25, R26, R27, R3: footprint Resistor_SMD:R_0805_2012Metric_Pad1.20x1.40mm_HandSolder -> Resistor_SMD:R_0402_1005Metric; LCSC Part # C17414 -> C25744
- R10, R11, R12, R9: footprint Resistor_SMD:R_0805_2012Metric_Pad1.20x1.40mm_HandSolder -> Resistor_SMD:R_0402_1005Metric; LCSC Part # (none) -> C11702
- R14, R15: footprint Resistor_SMD:R_0805_2012Metric_Pad1.20x1.40mm_HandSolder -> Resistor_SMD:R_0402_1005Metric; LCSC Part # C17710 -> C25117
- R16, R20, R4, R5, R7, R8: footprint Resistor_SMD:R_0805_2012Metric_Pad1.20x1.40mm_HandSolder -> Resistor_SMD:R_0402_1005Metric; LCSC Part # C17513 -> C11702
- R17, R18: footprint Resistor_SMD:R_0805_2012Metric_Pad1.20x1.40mm_HandSolder -> Resistor_SMD:R_0402_1005Metric; LCSC Part # C17596 -> C25100
- R2: footprint Resistor_SMD:R_0805_2012Metric_Pad1.20x1.40mm_HandSolder -> Resistor_SMD:R_0402_1005Metric; LCSC Part # C17634 -> C25105
- R21, R22: footprint Resistor_SMD:R_0805_2012Metric_Pad1.20x1.40mm_HandSolder -> Resistor_SMD:R_0402_1005Metric; LCSC Part # C17733 -> C25905
- R23: footprint Resistor_SMD:R_0805_2012Metric_Pad1.20x1.40mm_HandSolder -> Resistor_SMD:R_0402_1005Metric; LCSC Part # C17713 -> C25792
- R28: footprint Resistor_SMD:R_0805_2012Metric_Pad1.20x1.40mm_HandSolder -> Resistor_SMD:R_0402_1005Metric; LCSC Part # C17407 -> C25741
- SW1: footprint Button_Switch_THT:SW_PUSH_6mm -> Button_Switch_SMD:SW_Push_1P1T_XKB_TS-1187A; LCSC C17513 -> C318884; LCSC Part # C114217 -> C318884
- SW2: footprint Button_Switch_THT:SW_PUSH_6mm -> Button_Switch_SMD:SW_Push_1P1T_XKB_TS-1187A; LCSC C114217 -> C318884; LCSC Part # C114217 -> C318884
- SW3, SW4, SW5: footprint Button_Switch_THT:SW_PUSH_6mm -> Button_Switch_SMD:SW_Push_1P1T_XKB_TS-1187A; LCSC Part # C114217 -> C318884
- U3: LCSC Part # C5122557 -> C17337
- U5: LCSC Part # C42419115 -> C41378174
- U8, U9: LCSC Part # C5582 -> C87282
- Y1: LCSC Part # C9002 -> C5160143
Connections:
- net BC1_2: now also U5.40 (GPIO26/ADC0); no longer U5.41 (GPIO27/ADC1)
- net BDIR2: now also U5.41 (GPIO27/ADC1); no longer U5.40 (GPIO26/ADC0)
- net GND: now also J2.SH (Casing); no longer J2.10 (Casing)
- net MCU_CLK: now also U5.13 (GPIO9); no longer U5.16 (GPIO12)
- net MUX_B_CEN: now also U5.17 (GPIO13); no longer U5.36 (GPIO24)
- net MUX_C_CEN: now also U5.18 (GPIO14); no longer U5.37 (GPIO25)
- net MUX_MONO: now also U5.19 (GPIO15); no longer U5.43 (GPIO29/ADC3)
- net MUX_PAN: now also U5.16 (GPIO12); no longer U5.35 (GPIO23)
- net OLED_SCL: now also U5.43 (GPIO29/ADC3); no longer U5.28 (GPIO17)
- net OLED_SDA: now also U5.42 (GPIO28/ADC2); no longer U5.27 (GPIO16)
- net SD_Amp: now also U5.31 (GPIO19); no longer U5.13 (GPIO9)
- net SD_CLK: now also U5.36 (GPIO24); no longer U5.34 (GPIO22)
- net SD_CMD: now also U5.37 (GPIO25); no longer U5.42 (GPIO28/ADC2)
- net SD_DAT0: now also U5.32 (GPIO20); no longer U5.29 (GPIO18)
- net SD_DAT1: now also U5.33 (GPIO21); no longer U5.31 (GPIO19)
- net SD_DAT2: now also U5.34 (GPIO22); no longer U5.32 (GPIO20)
- net SD_DAT3: now also U5.35 (GPIO23); no longer U5.33 (GPIO21)
- net SW_NEXT: now also U5.27 (GPIO16); no longer U5.17 (GPIO13)
- net SW_PLAY: now also U5.28 (GPIO17); no longer U5.18 (GPIO14)
- net SW_PREV: now also U5.29 (GPIO18); no longer U5.19 (GPIO15)
