File: pico chiptune player.kicad_pcb (KiCad board)
At the start: 4 copper layers, 118 x 92 mm, 47 parts, among them J2 MicroSD, SW1 Play / Pause, SW2 Next, SW3 Previous, U1 AY-3-8910, U2 0.96"OLED_I2C, U3 PAM8302, U4 YM2149F, U5 PAM8302

Commit message: Refactor code structure for improved readability and maintainability
Parts:
- removed U5: PAM8302, TModules:PAM8302A_Module
- added C14: 1uF, Capacitor_SMD:C_0805_2012Metric_Pad1.18x1.45mm_HandSolder, B.Cu at (108.0, 61.6)
- added C15: 10uF, Capacitor_SMD:CP_Elec_4x5.4, F.Cu at (119.5, 63.5)
- added C16: 1uF, Capacitor_SMD:C_0805_2012Metric_Pad1.18x1.45mm_HandSolder, F.Cu at (105.5, 70.8)
- added J3: Speaker_L, Connector_JST:JST_PH_B2B-PH-K_1x02_P2.00mm_Vertical, F.Cu at (101.0, 54.5)
- added J4: Speaker_R, Connector_JST:JST_PH_B2B-PH-K_1x02_P2.00mm_Vertical, F.Cu at (114.0, 54.5)
- added R13: 10K, Resistor_SMD:R_0805_2012Metric_Pad1.20x1.40mm_HandSolder, F.Cu at (113.8, 64.1)
- C10, C3: footprint Capacitor_SMD:CP_Elec_3x5.4 -> Capacitor_SMD:C_0805_2012Metric_Pad1.18x1.45mm_HandSolder
- C13: value 100nF -> 1uF; moved to F.Cu
- C8: value 100nF -> 1uF
- U3: value PAM8302 -> PAM8403; footprint TModules:PAM8302A_Module -> Package_SO:SOIC-16_3.9x9.9mm_P1.27mm
- moved C13 18.5 mm to (116.2, 69.0)
- moved C8 17.5 mm to (108.0, 65.4)
- moved U3 11.6 mm to (108.0, 63.5)
Connections:
- C10 pad 2: /AMP2_IN -> /AMP_INR
- C3 pad 2: Net-(U3-A+) -> /AMP_INL
- U3 pad 1: GND -> /SPK_L+
- U3 pad 2: +5V -> GND
- U3 pad 3: /SD_Amp -> /SPK_L-
- U3 pad 4: GND -> +5V
- U3 pad 5: Net-(U3-A+) -> /SD_Amp
- U3 pad 6: unconnected-(U3-OUT+-Pad6) -> +5V
- U3 pad 7: unconnected-(U3-OUT--Pad7) -> /AMP_INL
Routing:
- net /AMP_INR: track 0.00 -> 34.1 mm, vias 0 -> 1
- net /AMP_INL: track 0.00 -> 30.8 mm, vias 0 -> 1
- net /SPK_R-: track 0.00 -> 10.9 mm
- net /SPK_L-: track 0.00 -> 8.92 mm, vias 0 -> 1
- net /SPK_L+: track 0.00 -> 7.62 mm
- net Net-(U3-A+): track 7.24 -> 0.00 mm
- net /AMP2_IN: track 7.24 -> 0.00 mm
- net /SPK_R+: track 0.00 -> 6.91 mm
- net /SD_Amp: track 70.9 -> 67.9 mm, vias 0 -> 1
- net GND: track 40.9 -> 42.9 mm, vias 19 -> 24
- net /AMP_VREF: track 0.00 -> 1.83 mm
- net +5V: track 24.5 -> 25.3 mm, vias 4 -> 7
