File: pico chiptune player.kicad_pcb (KiCad board)
At the start: 4 copper layers, 118 x 92 mm, 52 parts, among them J2 MicroSD, J3 Speaker_L, J4 Speaker_R, SW1 Play / Pause, SW2 Next, SW3 Previous, U1 AY-3-8910, U2 0.96"OLED_I2C, U3 PAM8403, U4 YM2149F

Commit message: sch, pcb, docs: fit YM2149F in both PSG sockets
U1 was specified as an AY-3-8910 while U4 was a YM2149F. Both share
CLOCK and the JP1 /SEL net, so bridging JP1 halved the clock on the
YM2149F only and put the two stereo channels an octave apart. Specify
both sockets as YM2149F so JP1 divides both chips together; document a
matched AY-3-8910 pair as an alternative with JP1 open.

Also relink PCB footprints U4, C9, C11, C12 and R9-R12 to their own
schematic symbols. They were copied from U1/C1/C2/R4 and still carried
those symbols' paths, which would cross-match parts on the next
"Update PCB from Schematic". Connectivity is unchanged.

Co-Authored-By: Claude Opus 5.5 <noreply@anthropic.com>
Claude-Session: https://claude.ai/code/session_01RJQvxUpHsHwrbMu8k2obTf
Parts:
- U1: value AY-3-8910 -> YM2149F
Changed lines of the file:
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@@
 		(company "MotionFxDesign")
 		(comment 1 "Terence Ang / MotionFxDesign")
-		(comment 2 "Hardware AY-3-8910 / YM2149 Chiptune Player")
+		(comment 2 "Hardware Dual YM2149F Chiptune Player")
 	)
 	(layers
@@
 			)
 		)
-		(property "Value" "AY-3-8910"
+		(property "Value" "YM2149F"
 			(at 8.84 23.91 270)
 			(layer "B.SilkS")
@@
 			)
 		)
-		(property "Description" "AY-3-8910 3-voice Programmable Sound Generator (PSG), 40-pin DIP"
+		(property "Description" "YM2149F 3-voice Programmable Sound Generator (PSG), 40-pin DIP"
 			(at 0 0 0)
 			(layer "F.Fab")
@@
 			)
 		)
-		(property "Description" "AY-3-8910 3-voice Programmable Sound Generator (PSG), 40-pin DIP"
+		(property "Description" "YM2149F 3-voice Programmable Sound Generator (PSG), 40-pin DIP"
 			(at 0 0 0)
 			(layer "F.Fab")
